Commit message: navigation nodes is created

File: rvrl_description/urdf/p3at/model.urdf (robot description, URDF)
Before this commit: robot robot, 13 links, 12 joints
Joints:
- removed joint scan_joint
- added joint lidar_joint: type fixed, parent base_link, child base_scan, origin xyz=-0.064 0 0.122 rpy=0 0 0

Commit message: Added sonar sensor to p3at model and added rvrl_tutorial directory

File: rvrl_description/urdf/p3at/model.urdf (robot description, URDF)
Before this commit: robot robot, 13 links, 12 joints
Links:
- added link front_sonar, mass 0.1
Joints:
- added joint base_front_joint: type fixed, parent base_link, child front_sonar, origin xyz=0.0 0 0.0 rpy=0 0 0
